File: Kicad/RHT device/RHT device.kicad_pcb (KiCad board)
At the start: 4 copper layers, 40 x 48.4 mm, 31 parts, among them IC1 PIC18LF14K50-I_SO, IC2 HTU20D, Q1 SMMBT5551LT1G, Q2 SMMBT5551LT1G, Q3 SMMBT5551LT1G, Q4 SMMBT5551LT1G, U1 CC56-12EWA, U2 CH075-2032

Commit message: New HW version 1.0
Parts:
- removed G***: LOGO, MDV:logo_MDV_3
- removed LED1: LTST-C171GKT, Library_Loader:LEDC2012X90N
- removed the R10 at (104.1, 60.7)
- removed the REF** at (137.7, 33.7)
- added REF**: OSHW-Logo2_14.6x12mm_SilkScreen, Symbol:OSHW-Logo2_14.6x12mm_SilkScreen, B.Cu at (132.1, 65.4)
- IC2: value HTU20D -> HPP845E034R5; footprint Library_Loader:SON50P250X250X100-9N-D -> User_lib:SON100P300X300X100-7N
- R3, R5, R7, R9: value 100 -> 220
- moved C2 0.25 mm to (120.8, 29.4)
- moved IC2 0.23 mm to (120.8, 26.6)
- renumbered C3 to C2, C2 to C3, ISCP to J1, R13 to R10, R14 to R11, R11 to R12, R12 to R13
Connections:
- IC1 pad 17: Net-(IC1-Pad17) -> unconnected-(IC1-VUSB-Pad17)
- IC2 pad 3: Net-(IC2-Pad3) -> unconnected-(IC2-NC_1-Pad3)
- IC2 pad 4: Net-(IC2-Pad4) -> unconnected-(IC2-NC_2-Pad4)
- J1 pad 6: Net-(J1-Pad6) -> unconnected-(J1-UNUSED/LVP-Pad6)
- R12 pad 1: Net-(R11-Pad1) -> Net-(R12-Pad1)
- R13 pad 1: Net-(R11-Pad1) -> Net-(R12-Pad1)
- S1 pad 1: Net-(R11-Pad1) -> gnd
- S1 pad 3: Net-(R11-Pad1) -> Net-(R12-Pad1)
- S1 pad 4: gnd -> Net-(R12-Pad1)
Routing:
- net Net-(R11-Pad1): track 51.8 -> 0.00 mm, vias 2 -> 0
- net Net-(R12-Pad1): track 0.00 -> 27.6 mm, vias 0 -> 2
- net gnd: track 138.3 -> 121.3 mm, vias 6 -> 5
- net /D_f: track 46.5 -> 33.2 mm
- net /D_g: track 29.7 -> 43.0 mm
- net /PGC: track 19.6 -> 10.5 mm, vias 0 -> 2
- net /CC_3: track 21.9 -> 29.4 mm, vias 0 -> 2
- net +3V: track 126.3 -> 132.7 mm, vias 4 -> 11
- net /I2C_DATA: track 65.5 -> 60.2 mm, vias 3 -> 4
- net /D_b: track 61.6 -> 56.7 mm, vias 2 -> 3
- net /I2C_SCK: track 81.8 -> 77.8 mm
- net /D_d: track 24.8 -> 28.5 mm, vias 1 -> 2
- net /CC_2: track 31.6 -> 34.4 mm, vias 0 -> 2
- net /B_1: track 22.9 -> 20.5 mm, vias 3 -> 4
- net /D_c: track 47.9 -> 50.0 mm, vias 2 -> 3
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- removed copper zone on In1.Cu, net +3V
- removed copper zone on In2.Cu, net gnd
Other:
- outline, holes or cut-outs redrawn
- copper layers 4 -> 2
- board text added: "Https://www.makingdevices.com"
- board text added: "RHT Device Rev 1.0 - 2023"
- board text removed: "Https://makingdevices.com"
- board text removed: "RHT Device Rev 0.1 - 2021"
