File: Kicad/RHT device/RHT device.kicad_sch (KiCad schematic)
At the start: 29 parts, among them IC1 PIC18LF14K50-I_SO, IC2 HTU20D, J1 TC2030-MCP-NL, Q1 SMMBT5551LT1G, Q2 SMMBT5551LT1G, Q3 SMMBT5551LT1G, Q4 SMMBT5551LT1G, U1 CC56-12EWA, U2 CH075-2032

Commit message: New HW version 1.0
Parts:
- removed IC2: HTU20D, SON50P250X250X100-9N-D, symbol Library_Loader:HTU20D
- removed LED1: LTST-C171GKT, LEDC2012X90N, symbol BytesCounter-rescue:LTST-C171GKT-SamacSys_Parts
- removed R10: 220, RESC2012X75N, symbol Library_Loader:ERJP6WF1303V
- added IC2: HPP845E034R5, SON100P300X300X100-7N, symbol SamacSys_Parts:HPP845E034R5
- R3, R5, R7, R9: value 100 -> 220
- renumbered C3 to C2, C2 to C3, R13 to R10, R14 to R11, R11 to R12, R12 to R13
Connections:
- net +3V: now also IC2.5 (VDD)
- net I2C_DATA: now also IC2.1 (DATA)
- net I2C_SCK: now also IC2.6 (SCK)
- net gnd: now also S1.1, IC2.2 (GND), IC2.7 (EP); no longer S1.4
- net at R12.1, R13.1, S1.3: now also S1.4; no longer S1.1
- no-connect marks 2 -> 4
Other:
- moved on the sheet: C2, S1
